File: hardware/test_pcb/ttc-map.kicad_pcb (KiCad board)
At the start: 2 copper layers, 42 x 57 mm, 29 parts, among them U1 TLC5947DAP

Commit message: add antenna keep out space
Parts:
- moved R2 38.9 mm to (89.0, 66.5), turned to 90 degrees
- moved R1 23.2 mm to (89.0, 69.0), turned to -90 degrees
Routing:
- net Net-(U1-BLANK): track 72.7 -> 95.3 mm, vias 0 -> 2
- net +3V3: track 86.6 -> 108.2 mm, vias 0 -> 3
- net /IREF: track 75.6 -> 88.4 mm
- net /LED16: track 45.1 -> 37.4 mm
- net /LED12: track 33.4 -> 27.4 mm
- net /LED17: track 46.6 -> 40.9 mm
- net /LED13: track 35.8 -> 30.2 mm
- net /LED18: track 48.0 -> 43.4 mm
- net /LED14: track 37.3 -> 33.0 mm
- net /LED15: track 39.7 -> 36.0 mm
- net GND: track 35.4 -> 32.6 mm, vias 25 -> 12
- net +5V: track 98.5 -> 95.7 mm
- net /LED19: track 66.5 -> 64.8 mm
- net Net-(U1-XLAT): track 51.1 -> 49.8 mm, vias 1 -> 2
